File: hw/sch_pcb/ISM01A.kicad_pcb (KiCad board)
At the start: 2 copper layers, 60.5 x 40.1 mm, 98 parts, among them J1 JUMP_3X2, J10 HEADER_2x01_PARALLEL, J11 HEADER_2x01_PARALLEL, J12 HEADER_2x01_PARALLEL, J13 HEADER_2x01_PARALLEL, J14 HEADER_2x01_PARALLEL, J15 HEADER_2x01_PARALLEL, J16 HEADER_2x01_PARALLEL, J17 HEADER_2x01_PARALLEL, J18 HEADER_2x01_PARALLEL, J19 HEADER_2x01_PARALLEL, J2 SMA, J20 HEADER_2x01_PARALLEL, J21 HEADER_2x01_PARALLEL, J22 HEADER_2x01_PARALLEL, J23 HEADER_2x01_PARALLEL, J24 HEADER_1x02, J25 HEADER_1x02, J26 HEADER_2x01_PARALLEL, J3 SMA, J4 JUMP_3X2, J6 HEADER_2x01_PARALLEL, J7 HEADER_2x01_PARALLEL, J8 HEADER_2x01_PARALLEL, J9 HEADER_2x01_PARALLEL, M1 HOLE, M2 HOLE, M3 HOLE, M4 HOLE, Q1 BC817, Q2 BC817, U1 LM1117, U2 Si1060-A-GM, Y1 ABS07-120-32.768KHZ, Y2 ABM3B-30.000MHZ-10-1-U-T

Commit message: Edit 3D model
Other:
- net class Default removed
- net class MLAB_power removed
