File: hw/sch_pcb/ISM01.kicad_pcb (KiCad board)
At the start: 2 copper layers, 60.5 x 40.1 mm, 98 parts, among them J1 JUMP_3X2, J10 HEADER_2x01_PARALLEL, J11 HEADER_2x01_PARALLEL, J12 HEADER_2x01_PARALLEL, J13 HEADER_2x01_PARALLEL, J14 HEADER_2x01_PARALLEL, J15 HEADER_2x01_PARALLEL, J16 HEADER_2x01_PARALLEL, J17 HEADER_2x01_PARALLEL, J18 HEADER_2x01_PARALLEL, J19 HEADER_2x01_PARALLEL, J2 SMA, J20 HEADER_2x01_PARALLEL, J21 HEADER_2x01_PARALLEL, J22 HEADER_2x01_PARALLEL, J23 HEADER_2x01_PARALLEL, J24 HEADER_1x02, J25 HEADER_1x02, J26 HEADER_2x01_PARALLEL, J3 SMA, J4 JUMP_3X2, J6 HEADER_2x01_PARALLEL, J7 HEADER_2x01_PARALLEL, J8 HEADER_2x01_PARALLEL, J9 HEADER_2x01_PARALLEL, M1 HOLE, M2 HOLE, M3 HOLE, M4 HOLE, Q1 BC817, Q2 BC817, U1 LM1117, U2 Si1060-A-GM, Y1 ABS07-120-32.768KHZ, Y2 ABM3B-30.000MHZ-10-1-U-T

Commit message: aktualizace na kicad 7
Parts:
- moved C13 173.4 mm to (159.2, 90.3)
- moved C21 173.4 mm to (163.0, 110.8)
- moved C22 173.4 mm to (155.0, 120.1)
- moved D1 173.4 mm to (130.8, 95.3)
- moved J2 173.4 mm to (178.5, 106.8)
- moved J20 173.4 mm to (155.0, 115.0)
- moved J24 173.4 mm to (163.7, 117.3)
- moved J26 173.4 mm to (144.8, 115.0)
- moved J3 173.4 mm to (178.5, 96.0)
- moved J8 173.4 mm to (146.7, 85.8)
- moved L10 173.4 mm to (156.9, 94.7)
- moved M2 173.4 mm to (178.5, 117.6)
- moved R16 173.4 mm to (155.0, 110.6)
- moved R4 173.4 mm to (146.7, 90.2)
- moved Y1 173.4 mm to (144.7, 96.0)
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Routing:
- net GND: track 321.6 -> 81.8 mm
