File: hw/sch_pcb/ISM01.kicad_sch (KiCad schematic)
At the start: 98 parts, among them J1 JUMP_3X2, J10 HEADER_2x01_PARALLEL, J11 HEADER_2x01_PARALLEL, J12 HEADER_2x01_PARALLEL, J13 HEADER_2x01_PARALLEL, J14 HEADER_2x01_PARALLEL, J15 HEADER_2x01_PARALLEL, J16 HEADER_2x01_PARALLEL, J17 HEADER_2x01_PARALLEL, J18 HEADER_2x01_PARALLEL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

Commit message: aktualizace na kicad 7
Other:
- note added: "Component values are optimised for 433MHz"
- note removed: "433MHz"
- title: NAME -> ISM01
